File: 9W LED driver.sch (KiCad schematic (older format))
At the start: 27 parts, among them IC1 Si 9752 680PY89

Commit message: refined design
Parts:
- IC1: value Si 9752 680PY89 -> SIC 9752 680PY89
Changed lines of the file:
@@
 P 7150 3250
 F 0 "IC1" H 7150 3815 50  0000 C CNN
-F 1 "Si 9752 680PY89" H 7150 3724 50  0000 C CNN
+F 1 "SIC 9752 680PY89" H 7150 3724 50  0000 C CNN
 F 2 "Package_SO:SOIC-8_3.9x4.9mm_P1.27mm" H 7150 3250 50  0001 C CNN
 F 3 "http://ww1.microchip.com/downloads/en/DeviceDoc/20005588A.pdf" H 7150 3250 50  0001 C CNN
