File: 9W LED driver.sch (KiCad schematic (older format))
At the start: 27 parts, among them IC1 Si 9752 680PY89

Commit message: Updated Schematics
Parts:
- removed IC1: Si 9752 680PY89, Package_SO:SOIC-8_3.9x4.9mm_P1.27mm, symbol LED~Driver:Si_9752
- added U1: Sic9752, Package_SO:SOIC-8_3.9x4.9mm_P1.27mm, symbol LED~Driver:Sic9752
Connections:
- net labels added: +ve_output, GNDS
- wire segments 89 -> 64

Commit message: Updated PCB Layout
Connections:
- net labels removed: -ve_Rail
- wire segments 64 -> 66
Other:
- moved on the sheet: C1, C4, H1, H2, L2, R5
Changed lines of the file:
@@
 L Mechanical:MountingHole_Pad H1
 U 1 1 63E3BE97
-P 6650 3450
-F 0 "H1" V 6604 3600 50  0000 L CNN
-F 1 "+ve Output" V 6695 3600 50  0000 L CNN
-F 2 "9W LED driver:Pad" H 6650 3450 50  0001 C CNN
-F 3 "~" H 6650 3450 50  0001 C CNN
-	1    6650 3450
+P 6550 3450
+F 0 "H1" V 6504 3600 50  0000 L CNN
+F 1 "+ve Output" V 6595 3600 50  0000 L CNN
+F 2 "9W LED driver:Pad" H 6550 3450 50  0001 C CNN
+F 3 "~" H 6550 3450 50  0001 C CNN
+	1    6550 3450
 	-1   0    0    1
 $EndComp
-Text GLabel 6650 3200 1    50   Input ~ 0
-+ve_output
-Wire Wire Line
-	6650 3350 6650 3200
-Wire Wire Line
-	6000 3200 6000 3300
-Wire Wire Line
-	6350 3200 6350 3300
-Text GLabel 6350 3200 1    50   Input ~ 0
-+ve_output
-Wire Wire Line
-	6000 3600 6000 3750
+Text GLabel 6550 3200 1    50   Input ~ 0
++ve_output
+Wire Wire Line
+	6550 3350 6550 3200
+Wire Wire Line
+	5900 3200 5900 3300
+Wire Wire Line
+	6250 3200 6250 3300
+Text GLabel 6250 3200 1    50   Input ~ 0
++ve_output
+Wire Wire Line
+	5900 3600 5900 3750
 $Comp
 L power:GNDS #PWR0101
 U 1 1 63E7B8A5
-P 6000 3750
-F 0 "#PWR0101" H 6000 3500 50  0001 C CNN
-F 1 "GNDS" H 6005 3577 50  0000 C CNN
-F 2 "" H 6000 3750 50  0001 C CNN
-F 3 "" H 6000 3750 50  0001 C CNN
-	1    6000 3750
+P 5900 3750
+F 0 "#PWR0101" H 5900 3500 50  0001 C CNN
+F 1 "GNDS" H 5905 3577 50  0000 C CNN
+F 2 "" H 5900 3750 50  0001 C CNN
+F 3 "" H 5900 3750 50  0001 C CNN
+	1    5900 3750
 	1    0    0    -1
 $EndComp
@@
 L Device:R R5
 U 1 1 63E5FD7D
-P 6350 3450
-F 0 "R5" V 6263 3377 50  0000 L CNN
-F 1 "R SMD 154" V 6460 3287 50  0000 L CNN
-F 2 "Resistor_SMD:R_0805_2012Metric" V 6280 3450 50  0001 C CNN
-F 3 "~" H 6350 3450 50  0001 C CNN
-	1    6350 3450
-	1    0    0    -1
-$EndComp
-Wire Wire Line
-	6350 3600 6350 3750
+P 6250 3450
+F 0 "R5" V 6163 3377 50  0000 L CNN
+F 1 "R SMD 154" V 6360 3287 50  0000 L CNN
+F 2 "Resistor_SMD:R_0805_2012Metric" V 6180 3450 50  0001 C CNN
+F 3 "~" H 6250 3450 50  0001 C CNN
+	1    6250 3450
+	1    0    0    -1
+$EndComp
+Wire Wire Line
+	6250 3600 6250 3750
 $Comp
 L power:GNDS #PWR0102
 U 1 1 63D9BBCF
-P 6350 3750
-F 0 "#PWR0102" H 6350 3500 50  0001 C CNN
-F 1 "GNDS" H 6355 3577 50  0000 C CNN
-F 2 "" H 6350 3750 50  0001 C CNN
-F 3 "" H 6350 3750 50  0001 C CNN
-	1    6350 3750
+P 6250 3750
+F 0 "#PWR0102" H 6250 3500 50  0001 C CNN
+F 1 "GNDS" H 6255 3577 50  0000 C CNN
+F 2 "" H 6250 3750 50  0001 C CNN
+F 3 "" H 6250 3750 50  0001 C CNN
+	1    6250 3750
 	1    0    0    -1
 $EndComp
@@
 L Mechanical:MountingHole_Pad H2
 U 1 1 63E3BE91
-P 5700 3500
-F 0 "H2" V 5654 3650 50  0000 L CNN
-F 1 "-ve Output" V 5745 3650 50  0000 L CNN
-F 2 "9W LED driver:Pad" H 5700 3500 50  0001 C CNN
-F 3 "~" H 5700 3500 50  0001 C CNN
-	1    5700 3500
+P 5600 3500
+F 0 "H2" V 5554 3650 50  0000 L CNN
+F 1 "-ve Output" V 5645 3650 50  0000 L CNN
+F 2 "9W LED driver:Pad" H 5600 3500 50  0001 C CNN
+F 3 "~" H 5600 3500 50  0001 C CNN
+	1    5600 3500
 	1    0    0    -1
 $EndComp
@@
 L power:GNDS #PWR0104
 U 1 1 63E77AAB
-P 5700 3750
-F 0 "#PWR0104" H 5700 3500 50  0001 C CNN
-F 1 "GNDS" H 5705 3577 50  0000 C CNN
-F 2 "" H 5700 3750 50  0001 C CNN
-F 3 "" H 5700 3750 50  0001 C CNN
-	1    5700 3750
-	1    0    0    -1
-$EndComp
-Wire Wire Line
-	5700 3750 5700 3600
+P 5600 3750
+F 0 "#PWR0104" H 5600 3500 50  0001 C CNN
+F 1 "GNDS" H 5605 3577 50  0000 C CNN
+F 2 "" H 5600 3750 50  0001 C CNN
+F 3 "" H 5600 3750 50  0001 C CNN
+	1    5600 3750
+	1    0    0    -1
+$EndComp
+Wire Wire Line
+	5600 3750 5600 3600
 $Comp
 L power:GNDS #PWR0105
@@
 Text GLabel 4700 2900 2    50   Input ~ 0
 +ve_output
-$Comp
-L pspice:INDUCTOR L2
-U 1 1 63F68F60
-P 4250 2900
-F 0 "L2" H 4204 3022 50  0000 L CNN
-F 1 "transformer" H 4295 3135 50  0000 C TNN
-F 2 "9W LED driver:Inductor_Transformer" H 4250 2900 50  0001 C CNN
-F 3 "~" H 4250 2900 50  0001 C CNN
-	1    4250 2900
-	1    0    0    -1
-$EndComp
 $Comp
 L Device:R R6
@@
 L Device:C C4
 U 1 1 63E5FD83
-P 6000 3450
-F 0 "C4" V 5869 3445 50  0000 C CNN
-F 1 "C 82uF 80V" V 6145 3465 50  0000 C CNN
-F 2 "Capacitor_THT:CP_Radial_D10.0mm_P7.50mm" H 6038 3300 50  0001 C CNN
-F 3 "~" H 6000 3450 50  0001 C CNN
-	1    6000 3450
+P 5900 3450
+F 0 "C4" V 5769 3445 50  0000 C CNN
+F 1 "C 82uF 80V" V 6045 3465 50  0000 C CNN
+F 2 "Capacitor_THT:CP_Radial_D10.0mm_P7.50mm" H 5938 3300 50  0001 C CNN
+F 3 "~" H 5900 3450 50  0001 C CNN
+	1    5900 3450
 	1    0    0    -1
 $EndComp
@@
 Wire Wire Line
 	3550 1700 4200 1700
-Text GLabel 3900 1400 0    50   Input ~ 0
--ve_Rail
 Wire Notes Line
 	5300 2150 700  2150
-$Comp
-L power:GNDS #PWR0103
-U 1 1 63D9411D
-P 5400 3750
-F 0 "#PWR0103" H 5400 3500 50  0001 C CNN
-F 1 "GNDS" H 5405 3577 50  0000 C CNN
-F 2 "" H 5400 3750 50  0001 C CNN
-F 3 "" H 5400 3750 50  0001 C CNN
-	1    5400 3750
-	1    0    0    -1
-$EndComp
-Wire Wire Line
-	5400 3750 5400 3600
-Text GLabel 5400 3600 1    50   Input ~ 0
--ve_Rail
-Text GLabel 6000 3200 1    50   Input ~ 0
-+ve_output
-Text GLabel 6950 3550 3    50   Input ~ 0
--ve_Rail
+Text GLabel 5900 3200 1    50   Input ~ 0
++ve_output
 Wire Notes Line
 	7250 4150 7250 2250
@@
 L Device:C C1
 U 1 1 63D908A6
-P 6950 3400
-F 0 "C1" V 6797 3343 50  0000 L CNN
-F 1 "CY400 473KE" V 7112 3355 50  0000 C CNN
-F 2 "Capacitor_THT:C_Rect_L11.0mm_W7.3mm_P10.00mm_MKT" H 6988 3250 50  0001 C CNN
-F 3 "~" H 6950 3400 50  0001 C CNN
-	1    6950 3400
-	1    0    0    -1
-$EndComp
-Text GLabel 6950 3100 1    50   Input ~ 0
+P 6850 3400
+F 0 "C1" V 6697 3343 50  0000 L CNN
+F 1 "CY400 473KE" V 7012 3355 50  0000 C CNN
+F 2 "Capacitor_THT:C_Rect_L11.0mm_W7.3mm_P10.00mm_MKT" H 6888 3250 50  0001 C CNN
+F 3 "~" H 6850 3400 50  0001 C CNN
+	1    6850 3400
+	1    0    0    -1
+$EndComp
+Text GLabel 6850 3100 1    50   Input ~ 0
 +ve_Rail
 Wire Wire Line
-	6950 3100 6950 3250
+	6850 3100 6850 3250
 Connection ~ 2500 3500
+$Comp
+L power:GNDS #PWR0103
+U 1 1 63D91799
+P 6850 3750
+F 0 "#PWR0103" H 6850 3500 50  0001 C CNN
+F 1 "GNDS" H 6855 3577 50  0000 C CNN
+F 2 "" H 6850 3750 50  0001 C CNN
+F 3 "" H 6850 3750 50  0001 C CNN
+	1    6850 3750
+	1    0    0    -1
+$EndComp
+Wire Wire Line
+	6850 3550 6850 3750
+$Comp
+L power:GNDS #PWR0106
+U 1 1 63D96773
+P 3750 1450
+F 0 "#PWR0106" H 3750 1200 50  0001 C CNN
+F 1 "GNDS" H 3755 1277 50  0000 C CNN
+F 2 "" H 3750 1450 50  0001 C CNN
+F 3 "" H 3750 1450 50  0001 C CNN
+	1    3750 1450
+	1    0    0    -1
+$EndComp
+Wire Wire Line
+	3900 1400 3750 1400
+Wire Wire Line
+	3750 1400 3750 1450
+$Comp
+L pspice:INDUCTOR L2
+U 1 1 63F68F60
+P 4250 2900
+F 0 "L2" H 4204 2738 50  0000 L CNN
+F 1 "transformer" H 4252 2856 50  0000 C TNN
+F 2 "9W LED driver:Inductor_Transformer" H 4250 2900 50  0001 C CNN
+F 3 "~" H 4250 2900 50  0001 C CNN
+	1    4250 2900
+	-1   0    0    1
+$EndComp
 $EndSCHEMATC
