File: 9W LED driver.kicad_pcb (KiCad board)
At the start: 2 copper layers, 50.6 x 21.8 mm, 27 parts, among them IC1 Sic9752

Commit message: Schematic Correction
Parts:
- renumbered + to H1, - to H2, IC1 to U1
Connections:
- C5 pad 1: Net-(C5-Pad1) -> Net-(C3-Pad1)
- L2 pad 2: Net-(C5-Pad1) -> Net-(C3-Pad1)
- R6 pad 2: Net-(C5-Pad1) -> Net-(C3-Pad1)
- U1 pad 2: Net-(C5-Pad1) -> Net-(C3-Pad1)
Routing:
- net Net-(C3-Pad1): track 15.9 -> 35.1 mm
- net Net-(C5-Pad1): track 15.1 -> 0.00 mm

Commit message: Fixed Schematic and Updated PCB
Parts:
- C1: value CY400 473KE -> 3.3uF 400V
- C2: value Ceramic 103 -> 0.01uF 400V
- C3: value C 4.7uF 50v -> 4.7uF 50V
- C4: value C 82uF 80V -> 82uF 80V
- C5: value C 100pF 50V -> 220nF 50V
- C6: value C 100pF 50V -> ~
- F1, F2: value R 56.00 ± 5% -> 56.00 ± 5%
- L1: value L 7mH NTL- -> 7mH
- L2: value transformer -> 2.1mH
- MOV1: value MOV-07D511K 320V 100pF 10% -> 320V 100pF
- R1, R2: value R SMD 334 -> 330K
- R10, R9: value R SMD 3R30 -> 3.3
- R3: value SMD 473 -> 47K
- R4: value R SMD 243 -> 24K
- R5, R6: value R SMD 154 -> 150K
- R7: value R SMD 211 -> 210
- R8: value R SMD 3R30 -> (none)
- moved C3 1.99 mm to (77.4, 69.1), turned to 0 degrees
- renumbered H1 to +, H2 to -
Connections:
- C3 pad 1: Net-(C3-Pad1) -> Net-(D1-K)
- C3 pad 2: Net-(C3-Pad2) -> Net-(U1-GND)
- C5 pad 1: Net-(C3-Pad1) -> Net-(U1-GND)
- D1 pad 1: Net-(C3-Pad2) -> Net-(D1-K)
- L2 pad 2: Net-(C3-Pad1) -> Net-(U1-GND)
- R10 pad 2: Net-(C3-Pad1) -> Net-(U1-GND)
- R2 pad 2: Net-(C3-Pad2) -> Net-(D1-K)
- R6 pad 2: Net-(C3-Pad1) -> Net-(U1-GND)
- R9 pad 2: Net-(C3-Pad1) -> Net-(U1-GND)
- U1 pad 2: Net-(C3-Pad1) -> Net-(U1-GND)
- U1 pad 3: Net-(C3-Pad2) -> Net-(D1-K)
Routing:
- net Net-(C3-Pad1): track 35.1 -> 0.00 mm
- net Net-(U1-GND): track 0.00 -> 34.9 mm
- net Net-(C3-Pad2): track 15.1 -> 0.00 mm
- net Net-(D1-K): track 0.00 -> 14.8 mm
Other:
- net class Default removed
